File: pcb/pcb.kicad_pcb (KiCad board)
At the start: 2 copper layers, 65 parts, among them J1 RJ45, J2 RJ45, SW1 Keyswitch, SW10 Keyswitch, SW11 Keyswitch, SW12 Keyswitch, SW13 Keyswitch, SW14 Keyswitch, SW15 Keyswitch, SW16 Keyswitch, SW17 Keyswitch, SW18 Keyswitch, SW19 Keyswitch, SW2 Keyswitch, SW20 Keyswitch, SW21 Keyswitch, SW22 Keyswitch, SW23 Keyswitch, SW24 Keyswitch, SW25 Keyswitch, SW26 Keyswitch, SW27 Keyswitch, SW28 Keyswitch, SW29 Keyswitch, SW3 Keyswitch, SW30 Keyswitch, SW4 Keyswitch, SW5 Keyswitch, SW6 Keyswitch, SW7 Keyswitch, SW8 Keyswitch, SW9 Keyswitch

Commit message: add pcb left hand layout
Parts:
- A1: moved to F.Cu
- moved SW3 177.7 mm to (158.4, 175.0)
- moved D3 176.6 mm to (167.9, 168.8)
- moved D8 172.2 mm to (206.6, 185.5), turned to -120 degrees
- moved SW7 166.7 mm to (195.9, 185.1), turned to -30 degrees
- moved D7 162.3 mm to (188.6, 174.1), turned to -105 degrees
- moved SW6 160.5 mm to (177.8, 177.6), turned to -15 degrees
- moved SW9 157.2 mm to (121.4, 150.0)
- moved D10 152.4 mm to (131.0, 139.1)
- moved D12 152.0 mm to (188.1, 145.0)
- moved SW11 152.0 mm to (178.6, 150.0)
- moved SW10 149.6 mm to (159.5, 150.2)
- moved D11 148.7 mm to (169.1, 143.8)
- moved SW2 147.9 mm to (83.3, 164.3)
- moved D2 146.7 mm to (92.9, 158.1)
- moved SW12 144.7 mm to (140.5, 126.4)
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
Commit message: change pcb diode placement
Parts:
- D1, D10, D11, D12, D13, D14, D15, D16, D17, D18, D19, D2, D20, D21, D22, D23, D24, D25, D26, D27, D28, D29, D3, D30, D31, D32, D4, D5, D6, D7, D8, D9: moved to F.Cu
- moved D16 64.4 mm to (140.0, 168.8), turned to 90 degrees
- moved D15 55.7 mm to (135.0, 168.8), turned to 90 degrees
- moved D29 54.4 mm to (308.5, 168.8), turned to 90 degrees
- moved D20 52.7 mm to (288.5, 168.8), turned to 90 degrees
- moved D13 51.5 mm to (130.0, 168.8), turned to 90 degrees
- moved D12 51.5 mm to (142.5, 168.8), turned to 90 degrees
- moved D9 48.9 mm to (127.5, 168.8), turned to 90 degrees
- moved D17 47.6 mm to (298.5, 168.8), turned to 90 degrees
- moved D30 44.8 mm to (311.0, 168.8), turned to 90 degrees
- moved D25 42.1 mm to (306.0, 168.8), turned to 90 degrees
- moved D1 40.3 mm to (120.0, 168.8), turned to 90 degrees
- moved D11 40.3 mm to (137.5, 168.8), turned to 90 degrees
- moved D21 39.2 mm to (301.0, 168.8), turned to 90 degrees
- moved D4 36.7 mm to (145.0, 168.8), turned to 90 degrees
- moved D32 36.5 mm to (283.5, 168.8), turned to 90 degrees
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Routing:
- net COL-1r: track 0.00 -> 122.3 mm
- net COL-2: track 0.00 -> 122.0 mm
- net COL-0r: track 0.00 -> 102.8 mm
- net COL-3: track 0.00 -> 97.1 mm
- net COL-1: track 0.00 -> 83.7 mm
- net Net-(D16-A): track 0.00 -> 71.8 mm, vias 0 -> 1
- net ROW-3: track 0.00 -> 65.8 mm
- net COL-0: track 0.00 -> 63.1 mm
- net Net-(D20-A): track 0.00 -> 62.9 mm
- net COL-2r: track 0.00 -> 60.9 mm
- net Net-(D29-A): track 0.00 -> 58.5 mm, vias 0 -> 1
- net Net-(D12-A): track 0.00 -> 55.8 mm
- net Net-(D15-A): track 0.00 -> 55.1 mm, vias 0 -> 1
- net Net-(D30-A): track 0.00 -> 53.6 mm
- net Net-(D17-A): track 0.00 -> 53.4 mm
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Other:
- board outline added: 288.1 x 85.7 mm

Commit message: add pcb screw holes
Connections:
- A1 pad 1: COL-0 -> unconnected-(A1-GPIO0-Pad1)
- A1 pad 10: ROW-3 -> unconnected-(A1-GPIO7-Pad10)_1
- A1 pad 11: ROW-4 -> unconnected-(A1-GPIO8-Pad11)_1
- A1 pad 12: ROW-5 -> unconnected-(A1-GPIO9-Pad12)_1
- A1 pad 14: ROW-6 -> ROW-0
- A1 pad 15: ROW-7 -> ROW-1
- A1 pad 16: unconnected-(A1-GPIO12-Pad16) -> ROW-5
- A1 pad 17: unconnected-(A1-GPIO13-Pad17)_1 -> ROW-4
- A1 pad 19: unconnected-(A1-GPIO14-Pad19) -> ROW-6
- A1 pad 2: COL-1 -> unconnected-(A1-GPIO1-Pad2)_1
- A1 pad 20: unconnected-(A1-GPIO15-Pad20)_1 -> ROW-7
- A1 pad 21: unconnected-(A1-GPIO16-Pad21)_1 -> COL-1
- A1 pad 22: unconnected-(A1-GPIO17-Pad22)_1 -> COL-0
- A1 pad 24: unconnected-(A1-GPIO18-Pad24)_1 -> COL-2
- A1 pad 25: unconnected-(A1-GPIO19-Pad25) -> COL-3
- A1 pad 26: unconnected-(A1-GPIO20-Pad26)_1 -> ROW-2
- A1 pad 27: unconnected-(A1-GPIO21-Pad27) -> ROW-3
- A1 pad 4: COL-2 -> unconnected-(A1-GPIO2-Pad4)_1
- A1 pad 5: COL-3 -> unconnected-(A1-GPIO3-Pad5)
- A1 pad 6: ROW-0 -> unconnected-(A1-GPIO4-Pad6)_1
- A1 pad 7: ROW-1 -> unconnected-(A1-GPIO5-Pad7)_1
- A1 pad 9: ROW-2 -> unconnected-(A1-GPIO6-Pad9)
- J1 pad 1: COL-0 -> COL-1
- J1 pad 2: COL-1 -> ROW-5
- J1 pad 3: COL-2 -> COL-0
- J1 pad 4: COL-3 -> ROW-4
- J1 pad 5: ROW-4 -> COL-3
- J1 pad 6: ROW-5 -> ROW-6
- J1 pad 7: ROW-6 -> COL-2
- J2 pad 1: COL-0r -> COL-1r
- J2 pad 2: COL-1r -> ROW-5r
- J2 pad 3: COL-2r -> COL-0r
- J2 pad 4: COL-3r -> ROW-4r
- J2 pad 5: ROW-4r -> COL-3r
- J2 pad 6: ROW-5r -> ROW-6r
- J2 pad 7: ROW-6r -> COL-2r
Routing:
- net COL-3: track 97.1 -> 311.1 mm
- net COL-2: track 122.0 -> 291.3 mm
- net COL-3r: track 49.0 -> 188.1 mm
- net COL-0: track 63.1 -> 202.0 mm
- net COL-2r: track 60.9 -> 196.3 mm
- net COL-1: track 83.7 -> 189.4 mm
- net ROW-5: track 0.00 -> 103.9 mm
- net ROW-4: track 0.00 -> 101.4 mm
- net ROW-6: track 0.00 -> 96.4 mm
- net ROW-7: track 0.00 -> 93.8 mm
- net ROW-4r: track 10.9 -> 85.0 mm
- net ROW-6r: track 2.50 -> 72.4 mm
- net ROW-7r: track 5.00 -> 74.8 mm
- net ROW-5r: track 19.3 -> 88.0 mm
- net COL-0r: track 102.8 -> 135.3 mm
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Other:
- outline, holes or cut-outs redrawn

Commit message: fix pcb holes
Parts:
- added REF**: MountingHole_2.5mm, MountingHole:MountingHole_2.5mm, F.Cu at (246.5, 192.9)
- added REF**: MountingHole_2.5mm, MountingHole:MountingHole_2.5mm, F.Cu at (300.0, 119.1)
- added REF**: MountingHole_2.5mm, MountingHole:MountingHole_2.5mm, F.Cu at (238.7, 146.4)
- added REF**: MountingHole_2.5mm, MountingHole:MountingHole_2.5mm, F.Cu at (110.7, 184.5)
- added REF**: MountingHole_2.5mm, MountingHole:MountingHole_2.5mm, F.Cu at (128.6, 119.1)
- added REF**: MountingHole_2.5mm, MountingHole:MountingHole_2.5mm, F.Cu at (182.2, 192.9)
- added REF**: MountingHole_2.5mm, MountingHole:MountingHole_2.5mm, F.Cu at (189.9, 146.4)
- added REF**: MountingHole_2.5mm, MountingHole:MountingHole_2.5mm, F.Cu at (317.9, 184.5)
Routing:
- net COL-0r: track 135.3 -> 132.5 mm
Other:
- outline, holes or cut-outs redrawn

Commit message: add pcb mouse bites
Parts:
- added mouse-bite-2mm-slot: VAL**, Panelization:mouse-bite-2mm-slot, F.Cu at (200.0, 130.0)
- added mouse-bite-2mm-slot: VAL**, Panelization:mouse-bite-2mm-slot, F.Cu at (200.0, 190.0)
- moved SW29 125.7 mm to (235.5, 225.5), turned to -90 degrees
- moved SW28 121.1 mm to (254.6, 225.5), turned to -90 degrees
- moved REF** 103.5 mm to (215.3, 198.1), turned to -90 degrees
- moved SW2 101.6 mm to (164.5, 225.5), turned to 90 degrees
- moved SW1 101.4 mm to (145.4, 225.5), turned to 90 degrees
- moved SW25 100.0 mm to (235.5, 206.4), turned to -90 degrees
- moved SW24 94.2 mm to (254.6, 206.4), turned to -90 degrees
- moved D26 86.2 mm to (231.0, 193.7), turned to 0 degrees
- moved D30 83.1 mm to (231.0, 191.2), turned to 0 degrees
- moved D29 80.0 mm to (231.0, 188.7), turned to 0 degrees
- moved REF** 77.1 mm to (207.0, 126.7), turned to -90 degrees
- moved D25 77.0 mm to (231.0, 186.2), turned to 0 degrees
- moved REF** 75.2 mm to (184.7, 198.1), turned to 90 degrees
- moved SW5 75.0 mm to (164.5, 206.4), turned to 90 degrees
- moved SW4 74.8 mm to (145.4, 206.4), turned to 90 degrees
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Other:
- board size 288.1 x 85.7 mm -> 173.5 x 140.5 mm
